File: TPS54331_EVA_Board.kicad_pcb (KiCad board)
At the start: 2 copper layers, 40.9 x 19.3 mm, 27 parts, among them IC2 TPS54331DR, J1 Conn_01x02_Pin, J2 Conn_01x02_Pin

Commit message: Update LCEDA Project
Parts:
- removed S1: SWITCH_SMTS102, kicad_lceda:SMTS-102
- added R10: 715R, Resistor_SMD:R_0603_1608Metric, F.Cu at (113.3, 85.3)
- added R11: 0R, Resistor_SMD:R_0603_1608Metric, F.Cu at (115.3, 87.7)
- added R7: 0R, Resistor_SMD:R_0603_1608Metric, F.Cu at (109.2, 87.7)
- added R8: 1.8K, Resistor_SMD:R_0603_1608Metric, F.Cu at (111.8, 85.3)
- added R9: 0R, Resistor_SMD:R_0603_1608Metric, F.Cu at (112.2, 87.7)
- R1: value 10.2K -> 10K
- moved R5 2.46 mm to (114.9, 85.3)
- moved C1 2.43 mm to (116.5, 85.3)
- moved C2 2.41 mm to (118.1, 85.3)
- moved C12 1.00 mm to (101.6, 84.5)
- moved C13 1.00 mm to (99.3, 79.9)
- moved C14 1.00 mm to (99.3, 84.5)
- moved C3 1.00 mm to (101.6, 79.9)
- moved D1 1.00 mm to (96.5, 81.8)
- moved R2 0.67 mm to (110.2, 85.3), turned to 90 degrees
- moved R1 0.64 mm to (108.6, 85.3)
- moved C11 0.62 mm to (107.0, 85.3)
- moved R3 0.54 mm to (104.7, 84.5)
- moved R4 0.54 mm to (104.7, 86.0)
Connections:
- D1 pad 2: Net-(D1-A) -> VCC
- R2 pad 1: Net-(IC2-VSENSE) -> Net-(R2-Pad1)
Routing:
- net Net-(IC2-VSENSE): track 5.66 -> 18.2 mm
- net Net-(R8-Pad1): track 0.00 -> 3.77 mm
- net Net-(R10-Pad1): track 0.00 -> 3.66 mm
- net Net-(IC2-COMP): track 7.80 -> 10.3 mm
- net Net-(R2-Pad1): track 0.00 -> 1.65 mm
- net +5V: track 25.1 -> 26.2 mm, vias 40 -> 42
- net GND: vias 129 -> 120
- removed copper zone on F.Cu, net Net-(D1-A)
Other:
- board text added: "3.3V 5V 12V"
- board text added: "Default"
- board text added: "Designed By Sakura Neko"
- board text added: "NEKO_BEC_3A"
- board text added: "POWER!"
- board text removed: "Designed By Bowen-Meng"
- board text removed: "ON OFF"
- board text removed: "POWER!!"
