File: TPS54331_EVA_Board.kicad_sch (KiCad schematic)
At the start: 26 parts, among them IC2 TPS54331DR, J1 Conn_01x02_Pin, J2 Conn_01x02_Pin

Commit message: Update LCEDA Project
Parts:
- removed S1: SWITCH_SMTS102, kicad_lceda:SMTS-102, symbol kicad_lceda:SWITCH_SMTS102
- added R10: 715R, Resistor_SMD:R_0603_1608Metric, symbol Device:R
- added R11, R7, R9: 0R, Resistor_SMD:R_0603_1608Metric, symbol Device:R
- added R8: 1.8K, Resistor_SMD:R_0603_1608Metric, symbol Device:R
- R1: value 10.2K -> 10K
Connections:
- net GND: now also R10.2, R8.2
- net VCC: now also D1.2 (A)
- net at IC2.5 (VSENSE), R1.2: now also R11.1, R7.1, R9.1; no longer R2.1
- new net: R8.1, R9.2
- new net: R10.1, R11.2
- new net: R2.1, R7.2
- no-connect marks 1 -> 0
Other:
- note added: "12V"
- note added: "3.3V"
- note added: "5V"
- moved on the sheet: C1, C2, D2, R1, R2, R5, R6
